File: Motor Driver/Motor Driver ASIC .kicad_sch (KiCad schematic)
At the start: 44 parts, among them Q1 IPTC011N08NM5ATMA1, Q2 NMOS

Commit message: PCB V0.1
Parts:
- removed C?: 4.7uF, symbol Device:C
- removed C?: 100nF, symbol Device:C
- removed C?: 10uF 100V, symbol Device:C
- removed D? (x2): D, symbol Device:D
- removed D? (x2): LED, symbol Device:LED
- removed F?: 45A, symbol Device:Fuse
- removed FB? (x2): Noise Suppr, symbol Device:FerriteBead_Small
- removed K?: RAYEX-L90A, Relay_THT:Relay_SPST_RAYEX-L90A, symbol Relay:RAYEX-L90A
- removed M?: Motor_DC_ALT, symbol Motor:Motor_DC_ALT
- removed Q1: IPTC011N08NM5ATMA1, symbol Device:Q_NMOS_GDS
- removed Q2: NMOS, symbol Device:Q_NMOS_GDS
- removed Q?: generic mmos, symbol Device:Q_NMOS_GDS
- removed R? (x3): 2.7k, symbol Device:R
- removed R?: 3.5k, symbol Device:R
- removed R?: 499k, symbol Device:R
- removed R?: 900, symbol Device:R
- removed R?: 45k, symbol Device:R
- removed R?: 10k, symbol Device:R
- removed R?: 22k, symbol Device:R
- removed R?: 24k, symbol Device:R
- removed Rsense: 0.001, symbol Device:R_Shunt
- removed TP?: OC, symbol Connector:TestPoint
- removed TP?: Rsense+, symbol Connector:TestPoint
- removed TP?: CurrSense, symbol Connector:TestPoint
- removed TP?: V_{ref}, symbol Connector:TestPoint
- removed TP?: OT, symbol Connector:TestPoint
- removed TP?: Rsense-, symbol Connector:TestPoint
- removed TP?: Temp, symbol Connector:TestPoint
- removed U? (x6): Opamp_Dual, symbol Device:Opamp_Dual
- removed U?: INA138, Package_TO_SOT_SMD:SOT-23-5, symbol Amplifier_Current:INA138
- removed U?: LM20BIM7, Package_TO_SOT_SMD:SOT-353_SC-70-5, symbol Sensor_Temperature:LM20BIM7
- removed U? (x2): REF196, symbol Reference_Voltage:REF196
- removed U?: ADP3625, symbol MySymbols:ADP3625
- added C1: 1uF, Capacitor_SMD:C_0603_1608Metric_Pad1.08x0.95mm_HandSolder, symbol Device:C_Small
- added C2: 1nF, Capacitor_SMD:C_0603_1608Metric_Pad1.08x0.95mm_HandSolder, symbol Device:C_Small
- added C4: 4.7uF, Capacitor_SMD:C_0603_1608Metric_Pad1.08x0.95mm_HandSolder, symbol Device:C_Small
- added C5, C6: C_{SNUBH}, Capacitor_SMD:C_0603_1608Metric_Pad1.08x0.95mm_HandSolder, symbol Device:C_Small
- added J1, J2: Conn_01x02_Male, Connector_PinHeader_1.27mm:PinHeader_1x02_P1.27mm_Vertical, symbol Connector:Conn_01x02_Male
- added J4: Screw_Terminal_01x02, TerminalBlock:TerminalBlock_bornier-2_P5.08mm, symbol Connector:Screw_Terminal_01x02
- added JP1: J_{DT}, Jumper:SolderJumper-2_P1.3mm_Open_RoundedPad1.0x1.5mm, symbol Jumper:Jumper_2_Open
- added M1: Motor_DC_ALT, Connector_Wire:SolderWire-1.5sqmm_1x02_P7.8mm_D1.7mm_OD3.9mm, symbol Motor:Motor_DC_ALT
- added NT1: NetTie_2, NetTie:NetTie-2_SMD_Pad2.0mm, symbol Device:NetTie_2
- added Q1, Q2: IAUA250N04S6N005, IFX-PG-HSOF-5-1-V:IFX-PG-HSOF-5-1-V, symbol MySymbols:IAUA250N04S6N005
- added R1: R_{DT}, Resistor_SMD:R_0603_1608Metric_Pad0.98x0.95mm_HandSolder, symbol Device:R_Small
- added R2: R_{G}_{H}, Resistor_SMD:R_0603_1608Metric_Pad0.98x0.95mm_HandSolder, symbol Device:R_Small
- added R3: R_{G}_{L}, Resistor_SMD:R_0603_1608Metric_Pad0.98x0.95mm_HandSolder, symbol Device:R_Small
- added R4, R5: C_{SNUBH}, Resistor_SMD:R_0603_1608Metric_Pad0.98x0.95mm_HandSolder, symbol Device:R_Small
- added TP1: V_{Gate_HI}, TestPoint:TestPoint_Pad_D1.0mm, symbol Connector:TestPoint_Probe
- added TP2: V_{Gate_LO}, TestPoint:TestPoint_Pad_D1.0mm, symbol Connector:TestPoint_Probe
- added TP3: V_{Drain}, TestPoint:TestPoint_Pad_D1.0mm, symbol Connector:TestPoint_Probe
- added U1: 2ED21824S06J, Package_SO:SO-14_3.9x8.65mm_P1.27mm, symbol MySymbols:2ED21824S06J
Connections:
- net GND: now also C1.2, C2.2, C6.2, J2.2 (Pin_2), JP1.1 (A), NT1.1, Q2.1 (S), Q2.2 (S), Q2.3 (S), Q2.4 (S), R1.2, U1. (V_{SS}), U1.5 (COM)
- new net: C4.1, U1.13 (V_{B})
- new net: C4.2, C5.2, M1.2 (-), Q1.1 (S), Q1.2 (S), Q1.3 (S), Q1.4 (S), Q2.6 (D), R5.1, TP3.1, U1.11 (V_{S})
- new net: C2.1, JP1.2 (B), R1.1, U1.4 (DT)
- new net: C6.1, R5.2
- new net: Q2.5 (G), R3.2, TP2.1
- new net: R2.1, U1.12 (HO)
- new net: Q1.5 (G), R2.2, TP1.1
- new net: C5.1, R4.2
- new net: R3.1, U1.6 (LO)
- new net: U1.10 (N.C.), U1.14 (N.C.), U1.9 (N.C.)
- new net +BATT: J4.1 (Pin_1), M1.1 (+), Q1.6 (D), R4.1
- new net -BATT: J4.2 (Pin_2), NT1.2
- new net H_{IN}: J1.1 (Pin_1), U1.1 (HIN)
- new net L_{IN}: J1.2 (Pin_2), U1.2 (LIN)
- new net VCC: C1.1, J2.1 (Pin_1), U1.7 (VCC)
Other:
- note added: "20V Max"
- note added: "R_{GE}=9.72Ω"
- note added: "Short for 400ns DT"
- note removed: "0.1% Resistors"
- note removed: "All resistors are 1%"
- note removed: "Buffer Input"
- note removed: "Buffer Output"
- note removed: "Ceramic"
- note removed: "Current Sense Amplifier"
- note removed: "Gain = 100 4.5V at Imax"
- note removed: "I_{max}=45A P_{max}=I_{max}^{2}*Rsense =2025*${7d56cc24-13dc-424e-9509-1fc8193a03a3:VALUE}=2.025W V_{Burden max}=45mV"
- note removed: "L_{m}=19nH R_{m}=16mΩ E_{m}=L_{m}*I^{2}/2"
- note removed: "MLCC"
- note removed: "Mosfet Overtemprature Protection"
- note removed: "Mosfet must have fast turn on time"
- note removed: "OverCurrent Protection"
- note removed: "Overtemprature Output"
- note removed: "P_{max}=1kW I_{max}~=45A"
- note removed: "P_{max}=32.4W"
- note removed: "Protection for the FETs avalanche diode"
- note removed: "R_{DS}_{on}_{(max)}=1.1mΩ P_{max}=0.0011*45^2=2.23 W Θ_{J}_{Ambient}=62 °C/W T_{J}_{Ambient}=T_{A}+Θ_{JA}*P_{MAX}=160.3 °C Θ_{J}_{case}=0.4 °C/W T_{J}_{case}=T_{A}+Θ_{JA}*P_{MAX}=22.9 °C"
- note removed: "Schmitt Trigger High Threshold 4.2V Hysteresis ~50mV Needs fast OpAmp"
- note removed: "Schmitt Trigger Threshold 300mV ~ 130 °C Hysteresis 500mV ~ 90 °C"
