File: Motor Driver/Motor Driver.kicad_sch (KiCad schematic)
At the start: 12 parts

Commit message: PCB V0.1
Parts:
- removed C?: C, symbol Device:C
- removed U? (x3): Opamp_Dual, symbol Device:Opamp_Dual
- added U? (x5): Opamp_Quad, symbol Device:Opamp_Quad
Connections:
- net +24V: now also U?.3 (+)
- net Current Sense: now also U?.7
- net PWM: now also U?.10 (+); no longer U?.2 (INA)
- net at D?.2 (K), M?.1 (+), R?.2: now also U?.2 (-)
- net at R?.1, R?.2: now also U?.6 (-)
- new net: U?.1, U?.5 (+)
- new net: U?.2 (INA), U?.8, U?.9 (-)
Other:
- note added: "E=L*I^2/2"
- note added: "R_{DS}_{on}_{(max)}=16mΩ P_{max}=0.016*45^2=32.4W Θ_{JA}_{case}=1.58 T_{J}_{case}=T_{A}+Θ_{JA}*P_{MAX}=2134.480 °C Θ_{JA}_{ambient}=65.2 T_{J}_{ambient}=T_{A}+Θ_{JA}*P_{MAX}=73.2 °C"
- note removed: "R_{DS}_{on}=16mΩ P_{max}=0.016*45^2=32.4W Θ_{JA}_{case}=1.58 Θ_{JA}_{ambient}=65.2 T_{J}=T_{A}+Θ_{JA}*P_{MAX}=73.2C"
- moved on the sheet: C?, D?, M?, R?, U?
