File: Parent/BMS.kicad_sch (KiCad schematic)
At the start: 22 parts, among them U3 MCP3008, U4 TL074, U5 TL074

Commit message: Worked on Parent - Move Workspace to cloud
Parts:
- removed U4, U5: TL074, symbol Amplifier_Operational:TL074
- added BT10, BT11, BT12, BT13, BT14, BT8, BT9: Battery_Cell, symbol Device:Battery_Cell
- added K1: ADW11, Relay_THT:Relay_1P1T_NO_10x24x18.8mm_Panasonic_ADW11xxxxW_THT, symbol Relay:ADW11
- added Q3: BS870, Package_TO_SOT_SMD:SOT-23, symbol Transistor_FET:BS870
- added R22: 3M, symbol Device:R
- added U4: A2982, Package_SO:SOIC-20W_7.5x12.8mm_P1.27mm, symbol Transistor_Array:A2982
- added U5: LM319, symbol Comparator:LM319
- added U6: INA139, Package_TO_SOT_SMD:SOT-23-5, symbol Amplifier_Current:INA139
Connections:
- net Batt+: now also BT8.1 (+), K1.3, K1.5, K1.6, U5.11 (V+)
- net Node1: now also BT13.2 (-), BT14.1 (+)
- net Node2: now also BT12.2 (-), BT13.1 (+)
- net Node3: now also BT11.2 (-), BT12.1 (+)
- net Node4: now also BT10.2 (-), BT11.1 (+)
- net Node5: now also BT10.1 (+), BT9.2 (-)
- net Node6: now also BT8.2 (-), BT9.1 (+)
- net Batt- renamed -BATT
- net -BATT: now also BT14.2 (-), R22.2, U5.6 (V-)
- new net: Q3.2 (S), R22.1
- new net: K1.1, Q3.3 (D)
Other:
- moved on the sheet: BT1, BT2, BT3, BT4, BT5, BT6, BT7, R11, R12, R13, R14, R15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
