File: Battery with Active BMS/Battery with Active BMS.kicad_pcb (KiCad board)
At the start: 2 copper layers, 512 x 95 mm, 62 parts, among them J1 Balancer Connector, J2 74651195R, J3 74651195R, Q1 IRFP7430PBF, Q2 IRFP7430PBF, U1 TLI4971A050T5UE0001XUMA1, U3 MCP3008, U4 TC4427CPA, U5 LM2574HVN-5

Commit message: Updated Active BMS and BOM
Parts:
- removed HS2: MOS Heatsink, Heatsink:Heatsink_Fischer_FK224xx2201_25x8.3mm
- added R27: 1M, Resistor_THT:R_Axial_DIN0207_L6.3mm_D2.5mm_P10.16mm_Horizontal, F.Cu at (237.0, 242.1)
- added R28: 1M, Resistor_THT:R_Axial_DIN0207_L6.3mm_D2.5mm_P10.16mm_Horizontal, F.Cu at (332.4, 242.3)
- added R29: 1M, Resistor_THT:R_Axial_DIN0207_L6.3mm_D2.5mm_P10.16mm_Horizontal, F.Cu at (319.9, 242.3)
- added R30: 1M, Resistor_THT:R_Axial_DIN0207_L6.3mm_D2.5mm_P10.16mm_Horizontal, F.Cu at (420.6, 242.3)
- added R31: 1M, Resistor_THT:R_Axial_DIN0207_L6.3mm_D2.5mm_P10.16mm_Horizontal, F.Cu at (408.1, 242.3)
- added R32: 1M, Resistor_THT:R_Axial_DIN0207_L6.3mm_D2.5mm_P10.16mm_Horizontal, F.Cu at (395.8, 242.3)
- added R33: 1M, Resistor_THT:R_Axial_DIN0207_L6.3mm_D2.5mm_P10.16mm_Horizontal, F.Cu at (461.6, 242.3)
- added R34: 1M, Resistor_THT:R_Axial_DIN0207_L6.3mm_D2.5mm_P10.16mm_Horizontal, F.Cu at (474.1, 242.3)
- added R35: 1M, Resistor_THT:R_Axial_DIN0207_L6.3mm_D2.5mm_P10.16mm_Horizontal, F.Cu at (486.6, 242.3)
- added R36: 1M, Resistor_THT:R_Axial_DIN0207_L6.3mm_D2.5mm_P10.16mm_Horizontal, F.Cu at (499.0, 242.3)
- A1: footprint Module:Arduino_Nano -> Module:Arduino_Nano_WithMountingHoles
- C3: footprint Capacitor_SMD:C_0805_2012Metric_Pad1.18x1.45mm_HandSolder -> Capacitor_SMD:C_1206_3216Metric_Pad1.33x1.80mm_HandSolder
- D1: value D_Schottky -> 1N5817
- HS1: value MOS Heatsink -> Heatsink_Pad_2Pin; footprint Heatsink:Heatsink_Fischer_FK224xx2201_25x8.3mm -> Heatsink:Heatsink_Fischer_SK104-STC-STIC_35x13mm_2xDrill2.5mm
- J1: footprint Connector_PinSocket_2.54mm:PinSocket_1x07_P2.54mm_Vertical -> Connector_JST:JST_EH_B7B-EH-A_1x07_P2.50mm_Vertical
- Q1, Q2: value IRFP7430PBF -> IPP015N04NGXKSA1; footprint Package_TO_SOT_THT:TO-247-3_Vertical -> Package_TO_SOT_THT:TO-220F-3_Vertical
- R1, R10, R2, R4, R6, R8: footprint Resistor_SMD:R_0805_2012Metric_Pad1.20x1.40mm_HandSolder -> Resistor_THT:R_Axial_DIN0207_L6.3mm_D2.5mm_P10.16mm_Horizontal; moved to F.Cu
- R25, R26: value 10 -> 3.3Ω
- R3: value 2M -> 1M; footprint Resistor_SMD:R_0805_2012Metric_Pad1.20x1.40mm_HandSolder -> Resistor_THT:R_Axial_DIN0207_L6.3mm_D2.5mm_P10.16mm_Horizontal; moved to F.Cu
- R5: value 3M -> 1M; footprint Resistor_SMD:R_0805_2012Metric_Pad1.20x1.40mm_HandSolder -> Resistor_THT:R_Axial_DIN0207_L6.3mm_D2.5mm_P10.16mm_Horizontal; moved to F.Cu
- R7: value 4M -> 1M; footprint Resistor_SMD:R_0805_2012Metric_Pad1.20x1.40mm_HandSolder -> Resistor_THT:R_Axial_DIN0207_L6.3mm_D2.5mm_P10.16mm_Horizontal; moved to F.Cu
- R9: value 5M -> 1M; footprint Resistor_SMD:R_0805_2012Metric_Pad1.20x1.40mm_HandSolder -> Resistor_THT:R_Axial_DIN0207_L6.3mm_D2.5mm_P10.16mm_Horizontal; moved to F.Cu
- moved U4 75.6 mm to (33.7, 238.3), turned to 0 degrees
- moved R26 64.1 mm to (43.4, 252.4)
- moved R25 54.4 mm to (47.0, 245.8), turned to 180 degrees
- moved R10 40.5 mm to (511.4, 242.3), turned to 0 degrees
- moved R7 38.0 mm to (433.0, 242.3)
- moved U1 37.2 mm to (528.0, 238.8)
- moved HS1 33.2 mm to (48.2, 267.4), turned to 90 degrees
- moved C1 32.4 mm to (336.8, 204.2), turned to -90 degrees
- moved R5 27.9 mm to (344.8, 242.3)
- moved Q1 27.3 mm to (51.4, 264.8)
- moved C2 26.9 mm to (332.8, 204.2), turned to -90 degrees
- moved R9 25.9 mm to (449.2, 242.3), turned to 0 degrees
- moved J3 17.0 mm to (8.30, 273.7)
- moved A1 16.7 mm to (274.4, 200.9)
- moved BT11 16.7 mm to (130.6, 254.1)
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Connections:
- A1 pad 11: unconnected-(A1-D8-Pad11) -> /M1
- A1 pad 12: unconnected-(A1-D9-Pad12) -> /M2
- A1 pad 5: /OCD1 -> /OCD2
- A1 pad 6: /OCD2 -> /OCD1
- A1 pad 7: /M2 -> unconnected-(A1-D4-Pad7)
- A1 pad 8: /M1 -> unconnected-(A1-D5-Pad8)
- R3 pad 2: /Cell3 -> Net-(R27-Pad1)
- R5 pad 2: /Cell4 -> Net-(R28-Pad1)
- R7 pad 2: /Cell5 -> Net-(R30-Pad1)
- R9 pad 2: /Cell6 -> Net-(R33-Pad1)
Routing:
- net +3.3V: track 0.00 -> 323.3 mm, vias 0 -> 2
- net /OCD2: track 0.00 -> 312.7 mm
- net /OCD1: track 0.00 -> 303.9 mm, vias 0 -> 1
- net /V_{REF}: track 0.00 -> 275.3 mm, vias 0 -> 1
- net /A_{AOUT}: track 0.00 -> 271.9 mm, vias 0 -> 1
- net +BATT: track 0.00 -> 234.6 mm, vias 0 -> 43
- net /M1: track 30.1 -> 246.7 mm
- net /M2: track 36.4 -> 239.4 mm
- net Net-(Q2-G): track 106.5 -> 0.00 mm
- net +5V: track 0.00 -> 90.3 mm, vias 0 -> 1
- net /Cell3: track 21.5 -> 100.4 mm
- net /Cell2: track 99.4 -> 175.2 mm
- net Net-(Q1-G): track 67.9 -> 0.00 mm
- net /Cell1: track 309.8 -> 353.2 mm, vias 0 -> 89
- net Net-(BT1-+): track 269.3 -> 231.5 mm, vias 0 -> 45
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- added copper zone on F.Cu, net +5V
- added copper zone on B.Cu, net +BATT
- added copper zone on F.Cu, net +BATT
- added copper zone on B.Cu, net -BATT
- added copper zone on F.Cu, net -BATT
- added copper zone on B.Cu, net /Cell1
- added copper zone on F.Cu, net /Cell1
- added copper zone on B.Cu, net Net-(BT1-+)
- added copper zone on F.Cu, net Net-(BT1-+)
- added copper zone on B.Cu, net Net-(BT1--)
- added copper zone on F.Cu, net Net-(BT1--)
- added copper zone on B.Cu, net Net-(BT10-+)
- added copper zone on F.Cu, net Net-(BT10-+)
- added copper zone on B.Cu, net Net-(BT3--)
- added copper zone on F.Cu, net Net-(BT3--)
- added copper zone on B.Cu, net Net-(BT5--)
- added copper zone on F.Cu, net Net-(BT5--)
- added copper zone on B.Cu, net Net-(Q1-S)
- added copper zone on F.Cu, net Net-(Q1-S)

Commit message: Updated Battery with Active BMS Schem&PCB&BOM
Parts:
- R26: moved to F.Cu
- moved R9 193.2 mm to (523.7, 64.1), turned to 180 degrees
- moved J3 186.5 mm to (36.9, 89.4)
- moved R1 186.0 mm to (211.6, 64.0)
- moved R2 186.0 mm to (199.1, 64.0)
- moved R33 185.0 mm to (511.4, 64.1), turned to 180 degrees
- moved R10 184.9 mm to (462.2, 64.1), turned to 180 degrees
- moved R27 182.5 mm to (278.1, 64.2)
- moved R3 182.5 mm to (290.5, 64.2)
- moved R4 182.5 mm to (265.7, 64.2)
- moved R34 179.9 mm to (499.1, 64.1), turned to 180 degrees
- moved R36 179.9 mm to (474.5, 64.1), turned to 180 degrees
- moved R6 179.8 mm to (332.3, 64.2)
- moved R29 179.8 mm to (344.7, 64.2)
- moved R28 179.8 mm to (357.1, 64.2)
- moved R5 179.8 mm to (369.5, 64.2)
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Connections:
- J1 pad 1: Net-(BT1-+) -> -BATT
- J1 pad 2: Net-(BT1--) -> /Cell1
- J1 pad 3: Net-(BT3--) -> Net-(BT10-+)
- J1 pad 5: Net-(BT10-+) -> Net-(BT3--)
- J1 pad 6: /Cell1 -> Net-(BT1--)
- J1 pad 7: -BATT -> Net-(BT1-+)
Routing:
- net +5V: track 90.3 -> 292.7 mm, vias 1 -> 2
- net Net-(U4-~{OUT_A}): track 14.7 -> 85.3 mm
- net /Cell2: track 175.2 -> 123.7 mm
- net /Cell6: track 239.5 -> 190.2 mm
- net Net-(BT10-+): track 134.5 -> 90.1 mm
- net /Cell3: track 100.4 -> 61.8 mm
- net Net-(BT5--): track 58.3 -> 26.1 mm
- net /Cell4: track 41.2 -> 56.9 mm
- net Net-(BT3--): track 106.9 -> 91.3 mm
- net /M1: track 246.7 -> 233.9 mm
- net Net-(U4-~{OUT_B}): track 0.00 -> 11.6 mm
- net /M2: track 239.4 -> 228.2 mm
- net /Cell5: track 114.1 -> 125.1 mm
- net /Cell1: track 353.2 -> 342.3 mm
- net Net-(BT1--): track 176.3 -> 167.5 mm
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- added copper zone on B.Cu, net GND
- added copper zone on F.Cu, net GND
Other:
- board size 512 x 95 mm -> 514.8 x 95 mm

Commit message: Motor Driver V1.0
Parts:
- removed A1: Arduino_Nano_v2.x, Module:Arduino_Nano_WithMountingHoles
- removed D1: 1N5817, Diode_THT:D_DO-15_P5.08mm_Vertical_KathodeUp
- removed HS1: Heatsink_Pad_2Pin, Heatsink:Heatsink_Fischer_SK104-STC-STIC_35x13mm_2xDrill2.5mm
- removed L1: 100uH, Inductor_THT:L_Radial_D10.5mm_P5.00mm_Abacron_AISR-01
- removed TH1, TH2, TH3, TH4, TH5, TH6: 100k, Connector_PinSocket_2.54mm:PinSocket_1x02_P2.54mm_Vertical
- added B1: 7461383, lib:M5 Screw Terminal, F.Cu at (41.9, 33.4)
- added B2: 7461383, lib:M5 Screw Terminal, F.Cu at (106.1, 143.4)
- added B3: 7461383, lib:M5 Screw Terminal, F.Cu at (106.1, 33.4)
- added B4: 7461383, lib:M5 Screw Terminal, F.Cu at (72.0, 33.4)
- added B5: 7461383, lib:M5 Screw Terminal, F.Cu at (41.9, 143.4)
- added B6: 7461383, lib:M5 Screw Terminal, F.Cu at (79.9, 135.4)
- added BT13: Battery_Cell, lib:21700, F.Cu at (235.2, 139.4)
- added BT14: Battery_Cell, lib:21700, F.Cu at (235.2, 117.4)
- added BT15: Battery_Cell, lib:21700, F.Cu at (235.2, 95.4)
- added BT16: Battery_Cell, lib:21700, F.Cu at (159.2, 139.4)
- added BT17: Battery_Cell, lib:21700, F.Cu at (159.2, 117.4)
- added BT18: Battery_Cell, lib:21700, F.Cu at (159.2, 95.4)
- added C5: Capacitor, Capacitor_SMD:C_0805_2012Metric_Pad1.18x1.45mm_HandSolder, F.Cu at (62.0, 46.9)
- added H1: MountingHole_Pad, MountingHole:MountingHole_5.3mm_M5_Pad_Via, F.Cu at (93.0, 147.0)
- added H10: MountingHole, MountingHole:MountingHole_2.5mm_Pad, F.Cu at (45.5, 150.0)
- added H11: MountingHole, MountingHole:MountingHole_2.5mm_Pad, F.Cu at (80.0, 18.0)
- added H12: MountingHole, MountingHole:MountingHole_2.5mm_Pad, F.Cu at (80.0, 101.0)
- added H2: MountingHole_Pad, MountingHole:MountingHole_5.3mm_M5_Pad_Via, F.Cu at (93.0, 101.0)
- added H3: MountingHole_Pad, MountingHole:MountingHole_5.3mm_M5_Pad_Via, F.Cu at (93.0, 21.0)
- added H4: MountingHole_Pad, MountingHole:MountingHole_5.3mm_M5_Pad_Via, F.Cu at (93.0, 67.0)
- added H5: MountingHole, MountingHole:MountingHole_2.5mm_Pad, F.Cu at (106.0, 150.0)
- added H6: MountingHole, MountingHole:MountingHole_2.5mm_Pad, F.Cu at (105.9, 18.0)
- added H7: MountingHole, MountingHole:MountingHole_2.5mm_Pad, F.Cu at (347.9, 18.4)
- added H8: MountingHole, MountingHole:MountingHole_2.5mm_Pad, F.Cu at (348.0, 150.1)
- added H9: MountingHole, MountingHole:MountingHole_2.5mm_Pad, F.Cu at (18.0, 18.0)
- added P1: 22-28-4033, Connector_PinHeader_2.54mm:PinHeader_2x02_P2.54mm_Vertical, F.Cu at (68.0, 109.5)
- added P2: 61300511121, Connector_PinHeader_2.54mm:PinHeader_2x05_P2.54mm_Vertical, F.Cu at (46.8, 62.4)
- added P3: 61300811121, Connector_PinHeader_2.54mm:PinHeader_2x09_P2.54mm_Vertical, F.Cu at (46.9, 80.6)
- added P4: TSW-106-07-L-D, Connector_PinHeader_2.54mm:PinHeader_2x06_P2.54mm_Vertical, F.Cu at (49.5, 117.3)
- added P5: 22-28-4033, Connector_PinHeader_2.54mm:PinHeader_2x02_P2.54mm_Vertical, F.Cu at (68.1, 38.5)
- added R37: Res2, Resistor_SMD:R_0805_2012Metric_Pad1.20x1.40mm_HandSolder, F.Cu at (71.7, 90.9)
- added R38: Res2, Resistor_SMD:R_0805_2012Metric_Pad1.20x1.40mm_HandSolder, F.Cu at (71.9, 88.4)
- added R39: Res2, Resistor_SMD:R_0805_2012Metric_Pad1.20x1.40mm_HandSolder, F.Cu at (62.5, 109.6)
- added R40: Res2, Resistor_SMD:R_0805_2012Metric_Pad1.20x1.40mm_HandSolder, F.Cu at (60.5, 109.6)
- added R41: 1M, Resistor_THT:R_Axial_DIN0207_L6.3mm_D2.5mm_P10.16mm_Horizontal, F.Cu at (18.5, 73.8)
- added R42: 1M, Resistor_THT:R_Axial_DIN0207_L6.3mm_D2.5mm_P10.16mm_Horizontal, F.Cu at (21.5, 86.3)
- added R43: 1M, Resistor_THT:R_Axial_DIN0207_L6.3mm_D2.5mm_P10.16mm_Horizontal, F.Cu at (30.5, 111.3)
- added R44: 1M, Resistor_THT:R_Axial_DIN0207_L6.3mm_D2.5mm_P10.16mm_Horizontal, F.Cu at (27.5, 98.8)
- added R45: 4.7k, Resistor_SMD:R_0805_2012Metric_Pad1.20x1.40mm_HandSolder, F.Cu at (63.7, 56.3)
- added R46: 4.7k, Resistor_SMD:R_0805_2012Metric_Pad1.20x1.40mm_HandSolder, F.Cu at (69.7, 56.3)
- added R47: 1M, Resistor_THT:R_Axial_DIN0207_L6.3mm_D2.5mm_P10.16mm_Horizontal, F.Cu at (24.5, 86.3)
- added R48: 1M, Resistor_THT:R_Axial_DIN0207_L6.3mm_D2.5mm_P10.16mm_Horizontal, F.Cu at (21.5, 73.8)
- added R49: 1M, Resistor_THT:R_Axial_DIN0207_L6.3mm_D2.5mm_P10.16mm_Horizontal, F.Cu at (18.5, 61.4)
- added R50: 4.7k, Resistor_SMD:R_0805_2012Metric_Pad1.20x1.40mm_HandSolder, F.Cu at (69.7, 65.3)
- added R51: 4.7k, Resistor_SMD:R_0805_2012Metric_Pad1.20x1.40mm_HandSolder, F.Cu at (63.7, 65.3)
- added R52: 4.7k, Resistor_SMD:R_0805_2012Metric_Pad1.20x1.40mm_HandSolder, F.Cu at (58.1, 56.3)
- added R53: 4.7k, Resistor_SMD:R_0805_2012Metric_Pad1.20x1.40mm_HandSolder, F.Cu at (58.1, 65.3)
- added R61: 4.7k, Resistor_SMD:R_0805_2012Metric_Pad1.20x1.40mm_HandSolder, F.Cu at (52.1, 56.3)
- added R63: 4.7k, Resistor_SMD:R_0805_2012Metric_Pad1.20x1.40mm_HandSolder, F.Cu at (52.1, 65.3)
- added U11: EL817, Package_DIP:DIP-4_W7.62mm, F.Cu at (70.5, 70.6)
- added U16: EL817, Package_DIP:DIP-4_W7.62mm, F.Cu at (58.9, 61.5)
- added U17: EL817, Package_DIP:DIP-4_W7.62mm, F.Cu at (58.9, 70.5)
- added U2: ARDUINO_PRO_MINI, lib:MODULE_ARDUINO_PRO_MINI, F.Cu at (60.7, 90.9)
- added U8: EL817, Package_DIP:DIP-4_W7.62mm, F.Cu at (70.5, 61.6)
- BT1, BT10, BT11, BT12, BT2, BT3, BT4, BT5, BT6, BT7, BT8, BT9: footprint Battery:BatteryHolder_MPD_BH-18650-PC2 -> lib:21700
- C1: value 100nF -> Capacitor
- C2: value 22uF -> Capacitor; footprint Capacitor_SMD:CP_Elec_5x5.8 -> Capacitor_SMD:C_0805_2012Metric_Pad1.18x1.45mm_HandSolder
- C3: value 10n -> Capacitor; footprint Capacitor_SMD:C_1206_3216Metric_Pad1.33x1.80mm_HandSolder -> Capacitor_SMD:C_0805_2012Metric_Pad1.18x1.45mm_HandSolder
- C4: value 220uF -> Capacitor; footprint Capacitor_SMD:CP_Elec_6.3x5.8 -> Capacitor_SMD:C_0805_2012Metric_Pad1.18x1.45mm_HandSolder
- J1: value Balancer Connector -> B7B-EH-A(LF)(SN)
- J2, J3: value 74651195R -> B7B-EH-A(LF)(SN); footprint TerminalBlock_Wuerth:Wuerth_REDCUBE-THR_WP-THRSH_74651195_THR -> Connector_JST:JST_EH_B6B-EH-A_1x06_P2.50mm_Vertical
- Q1, Q2: value IPP015N04NGXKSA1 -> NMOS; footprint Package_TO_SOT_THT:TO-220F-3_Vertical -> lib:IAUA250N04S6N005AUMA1
- R1, R2, R28, R29, R35, R36: value 1M -> Res2; footprint Resistor_THT:R_Axial_DIN0207_L6.3mm_D2.5mm_P10.16mm_Horizontal -> Resistor_SMD:R_0805_2012Metric_Pad1.20x1.40mm_HandSolder
- R11, R13, R14, R15: value 220 -> 1M; footprint Resistor_SMD:R_0805_2012Metric_Pad1.20x1.40mm_HandSolder -> Resistor_THT:R_Axial_DIN0207_L6.3mm_D2.5mm_P10.16mm_Horizontal; moved to F.Cu
- R12, R16, R17, R18: value 220 -> Res2; moved to F.Cu
- R19, R20, R21, R24: value 100k -> Res2; moved to F.Cu
- R22, R23: value 100k -> 1M; footprint Resistor_SMD:R_0805_2012Metric_Pad1.20x1.40mm_HandSolder -> Resistor_THT:R_Axial_DIN0207_L6.3mm_D2.5mm_P10.16mm_Horizontal; moved to F.Cu
- R25: value 3.3Ω -> 1M; footprint Resistor_SMD:R_0805_2012Metric_Pad1.20x1.40mm_HandSolder -> Resistor_THT:R_Axial_DIN0207_L6.3mm_D2.5mm_P10.16mm_Horizontal; moved to F.Cu
- R26: value 3.3Ω -> Res2; footprint Resistor_SMD:R_0805_2012Metric_Pad1.20x1.40mm_HandSolder -> Resistor_THT:R_Axial_DIN0207_L6.3mm_D2.5mm_P10.16mm_Horizontal
- R27: value 1M -> Res2
- U1: value TLI4971A050T5UE0001XUMA1 -> TLI4971
- U3: value MCP3008 -> MPC3008; footprint Package_DIP:DIP-16_W7.62mm_LongPads -> Package_DIP:DIP-16_W7.62mm
- U4: value TC4427CPA -> TC4428CPA; footprint Package_DIP:DIP-8_W7.62mm_LongPads -> Package_DIP:DIP-8_W7.62mm
- U5: value LM2574HVN-5 -> LM78M05CT/NOPB; footprint Package_DIP:DIP-8_W7.62mm -> Connector_PinSocket_2.54mm:PinSocket_1x03_P2.54mm_Vertical
- moved J2 521.8 mm to (19.8, 149.9), turned to 0 degrees
- moved R9 504.4 mm to (24.5, 136.3), turned to -90 degrees
- moved R33 494.1 mm to (18.5, 98.8), turned to -90 degrees
- moved R34 481.1 mm to (18.5, 86.3), turned to -90 degrees
- moved U1 469.9 mm to (60.9, 36.2), turned to 90 degrees
- moved R10 441.7 mm to (24.5, 123.8), turned to -90 degrees
- moved R7 427.1 mm to (27.5, 136.3), turned to -90 degrees
- moved R30 423.8 mm to (18.5, 136.3), turned to -90 degrees
- moved R35 416.2 mm to (71.8, 95.9)
- moved R31 409.5 mm to (18.5, 123.8), turned to -90 degrees
- moved R36 403.8 mm to (71.8, 93.4)
- moved R32 395.6 mm to (18.5, 111.3), turned to -90 degrees
- moved R8 376.1 mm to (27.5, 123.8), turned to -90 degrees
- moved BT1 371.2 mm to (159.2, 29.4), turned to -90 degrees
- moved BT2 371.1 mm to (159.2, 51.4), turned to -90 degrees
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Connections:
- BT10 pad 2: /Cell1 -> Net-(BT10--)
- BT11 pad 1: /Cell1 -> Net-(BT10-+)
- BT11 pad 2: -BATT -> Net-(BT10--)
- BT12 pad 1: /Cell1 -> Net-(BT10-+)
- BT12 pad 2: -BATT -> Net-(BT10--)
- BT3 pad 1: Net-(BT1--) -> Net-(BT1-+)
- BT3 pad 2: Net-(BT3--) -> Net-(BT1--)
- BT4 pad 1: Net-(BT1--) -> Net-(BT4-+)
- BT4 pad 2: Net-(BT3--) -> Net-(BT1-+)
- BT5 pad 1: Net-(BT3--) -> Net-(BT4-+)
- BT5 pad 2: Net-(BT5--) -> Net-(BT1-+)
- BT6 pad 1: Net-(BT3--) -> Net-(BT4-+)
- BT6 pad 2: Net-(BT5--) -> Net-(BT1-+)
- BT7 pad 1: Net-(BT5--) -> Net-(BT10--)
- BT7 pad 2: Net-(BT10-+) -> Net-(BT4-+)
- BT8 pad 1: Net-(BT5--) -> Net-(BT10--)
- BT8 pad 2: Net-(BT10-+) -> Net-(BT4-+)
- BT9 pad 1: Net-(BT10-+) -> Net-(BT10--)
- BT9 pad 2: /Cell1 -> Net-(BT4-+)
- C1 pad 1: +BATT -> /OCD2
- C1 pad 2: -BATT -> GND
- C2 pad 1: +BATT -> /OCD1
- C2 pad 2: -BATT -> GND
- C3 pad 1: +5V -> +3.3V
- C3 pad 2: -BATT -> GND
- C4 pad 1: +5V -> /VREF
- C4 pad 2: -BATT -> GND
- J1 pad 1: -BATT -> Net-(BT16-+)
- J1 pad 2: /Cell1 -> Net-(BT13-+)
- J1 pad 4: Net-(BT5--) -> Net-(BT10--)
- J1 pad 5: Net-(BT3--) -> Net-(BT4-+)
- J1 pad 6: Net-(BT1--) -> Net-(BT1-+)
- J1 pad 7: Net-(BT1-+) -> Net-(BT1--)
- J2 pad 1: +BATT -> Net-(J2-Pad1)
- J3 pad 1: GND -> Net-(BT16-+)
- Q1 pad 1: Net-(Q1-G) -> GND
- Q1 pad 2: -BATT -> Net-(Q1-G)
- Q2 pad 1: Net-(Q2-G) -> Net-(Q2-D)
- Q2 pad 2: GND -> Net-(Q2-G)
- R1 pad 1: Net-(BT10-+) -> /OCD1
- R1 pad 2: /Cell2 -> +3.3V
- R10 pad 1: /Cell6 -> Net-(R10-Pad1)
- R10 pad 2: -BATT -> Net-(R10-Pad2)
- R11 pad 1: /Cell1 -> Net-(R11-Pad1)
- R11 pad 2: Net-(U3-CH0) -> Net-(R10-Pad1)
- R12 pad 1: /Cell2 -> /AOUT
- R12 pad 2: Net-(U3-CH1) -> Net-(U3-CH0)
- R13 pad 1: /Cell3 -> /Cell4
- R13 pad 2: Net-(U3-CH2) -> Net-(R11-Pad1)
- R14 pad 1: /Cell4 -> Net-(R14-Pad1)
- R14 pad 2: Net-(U3-CH3) -> /Cell3
- R15 pad 1: /Cell5 -> Net-(R15-Pad1)
- R15 pad 2: Net-(U3-CH4) -> Net-(J2-Pad2)
- R16 pad 1: /Cell6 -> /VREF
- R16 pad 2: Net-(U3-CH5) -> Net-(U3-CH1)
- R17 pad 1: /A_{AOUT} -> /Cell6
- R17 pad 2: Net-(U3-CH6) -> Net-(U3-CH2)
- R18 pad 1: /V_{REF} -> /Cell5
- R18 pad 2: Net-(U3-CH7) -> Net-(U3-CH3)
- R19 pad 1: -BATT -> /Cell4
- R19 pad 2: Net-(A1-A0) -> Net-(U3-CH4)
- R2 pad 1: /Cell2 -> /OCD2
- R2 pad 2: -BATT -> +3.3V
- R20 pad 1: -BATT -> /Cell3
- R20 pad 2: Net-(A1-A1) -> Net-(U3-CH5)
- R21 pad 1: -BATT -> /Cell2
- R21 pad 2: Net-(A1-A2) -> Net-(U3-CH6)
- R22 pad 1: -BATT -> Net-(R22-Pad1)
- R22 pad 2: Net-(A1-A3) -> Net-(R15-Pad1)
- R23 pad 1: -BATT -> Net-(R23-Pad1)
- R23 pad 2: Net-(A1-A4) -> Net-(R22-Pad1)
- R24 pad 1: -BATT -> /Cell1
- R24 pad 2: Net-(A1-A5) -> Net-(U3-CH7)
- R25 pad 1: Net-(Q1-G) -> Net-(R25-Pad1)
- R25 pad 2: Net-(U4-~{OUT_B}) -> Net-(R23-Pad1)
- R26 pad 1: Net-(Q2-G) -> GND
- R26 pad 2: Net-(U4-~{OUT_A}) -> Net-(U2-D9)
- R27 pad 1: Net-(R27-Pad1) -> GND
- R27 pad 2: /Cell3 -> Net-(U2-D8)
- R28 pad 1: Net-(R28-Pad1) -> Net-(Q1-G)
- R28 pad 2: Net-(R28-Pad2) -> Net-(U4B-OUTB)
- R29 pad 1: Net-(R28-Pad2) -> Net-(Q2-G)
- R29 pad 2: /Cell4 -> Net-(U4A-~{OUTA})
- R3 pad 1: Net-(BT5--) -> Net-(J2-Pad6)
- R3 pad 2: Net-(R27-Pad1) -> /Cell1
- R30 pad 2: Net-(R30-Pad2) -> Net-(J2-Pad1)
- R31 pad 1: Net-(R30-Pad2) -> Net-(R31-Pad1)
- R31 pad 2: Net-(R31-Pad2) -> Net-(R30-Pad1)
- R32 pad 1: Net-(R31-Pad2) -> Net-(R32-Pad1)
- R32 pad 2: /Cell5 -> Net-(R31-Pad1)
- R33 pad 2: Net-(R33-Pad2) -> Net-(R32-Pad1)
- R34 pad 1: Net-(R33-Pad2) -> Net-(R34-Pad1)
- R34 pad 2: Net-(R34-Pad2) -> Net-(R33-Pad1)
- R35 pad 1: Net-(R34-Pad2) -> GND
- R35 pad 2: Net-(R35-Pad2) -> /A0
- R36 pad 1: Net-(R35-Pad2) -> GND
- R36 pad 2: /Cell6 -> /A1
- R4 pad 1: /Cell3 -> GND
- R4 pad 2: -BATT -> /Cell1
- R5 pad 1: Net-(BT3--) -> Net-(R5-Pad1)
- R5 pad 2: Net-(R28-Pad1) -> Net-(J2-Pad5)
- R6 pad 1: /Cell4 -> /Cell2
- R6 pad 2: -BATT -> Net-(R5-Pad1)
- R7 pad 1: Net-(BT1--) -> Net-(R7-Pad1)
- R7 pad 2: Net-(R30-Pad1) -> Net-(J2-Pad4)
- R8 pad 1: /Cell5 -> Net-(R14-Pad1)
- R8 pad 2: -BATT -> Net-(R7-Pad1)
- R9 pad 1: Net-(BT1-+) -> Net-(R10-Pad2)
- R9 pad 2: Net-(R33-Pad1) -> Net-(J2-Pad3)
- U1 pad 2: -BATT -> GND
- U1 pad 3: /V_{REF} -> /VREF
- U1 pad 4: /A_{AOUT} -> /AOUT
- U1 pad 7: +BATT -> Net-(U1-IP-)
- U1 pad 8: Net-(BT1-+) -> Batt+
- U3 pad 11: /D_{IN} -> /DIN
- U3 pad 12: /D_{OUT} -> /DOUT
- U3 pad 14: -BATT -> GND
- U3 pad 15: +5V -> +3.3V
- U3 pad 16: +5V -> +3.3V
- U3 pad 9: -BATT -> GND
- U4 pad 1: (no net) -> unconnected-(U4C-NC-Pad1)
- U4 pad 2: /M2 -> Net-(U2-D8)
- U4 pad 3: -BATT -> GND
- U4 pad 4: /M1 -> Net-(U2-D9)
- U4 pad 5: Net-(U4-~{OUT_B}) -> Net-(U4B-OUTB)
- U4 pad 6: +5V -> +3.3V
- U4 pad 7: Net-(U4-~{OUT_A}) -> Net-(U4A-~{OUTA})
- U4 pad 8: (no net) -> unconnected-(U4C-NC-Pad8)
- U5 pad 1: +5V -> Batt+
- U5 pad 2: -BATT -> GND
- U5 pad 3: -BATT -> +3.3V
Routing:
- net /OCD2: track 312.7 -> 17.8 mm
- net +5V: track 292.7 -> 0.00 mm, vias 2 -> 0
- net /OCD1: track 303.9 -> 16.8 mm, vias 1 -> 0
- net /V_{REF}: track 275.3 -> 0.00 mm, vias 1 -> 0
- net /A_{AOUT}: track 271.9 -> 0.00 mm, vias 1 -> 0
- net -BATT: track 267.4 -> 0.00 mm, vias 142 -> 0
- net /Cell1: track 342.3 -> 81.7 mm, vias 89 -> 0
- net Net-(BT10--): track 0.00 -> 251.5 mm
- net +BATT: track 234.6 -> 0.00 mm, vias 43 -> 0
- net /M1: track 233.9 -> 0.00 mm
- net /M2: track 228.2 -> 0.00 mm
- net Net-(BT4-+): track 0.00 -> 173.7 mm
- net /Cell6: track 190.2 -> 20.3 mm
- net Net-(BT1--): track 167.5 -> 18.6 mm, vias 94 -> 0
- net Net-(BT1-+): track 235.4 -> 101.2 mm, vias 45 -> 0
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- added copper zone on B.Cu, net /Copper Conn 1
- added copper zone on F.Cu, net /Copper Conn 1
- added copper zone on B.Cu, net /Copper Conn 2
- added copper zone on F.Cu, net /Copper Conn 2
- added copper zone on B.Cu, net Batt+
- added copper zone on F.Cu, net Batt+
- added copper zone on B.Cu, net Net-(BT10--)
- added copper zone on F.Cu, net Net-(BT10--)
- added copper zone on B.Cu, net Net-(BT13-+)
- added copper zone on F.Cu, net Net-(BT13-+)
- added copper zone on B.Cu, net Net-(BT16-+)
- added copper zone on F.Cu, net Net-(BT16-+)
- added copper zone on B.Cu, net Net-(BT4-+)
- added copper zone on F.Cu, net Net-(BT4-+)
- added copper zone on F.Cu, net Net-(Q2-D)
- added copper zone on B.Cu, net Net-(U1-IP-)
- added copper zone on F.Cu, net Net-(U1-IP-)
- removed copper zone on F.Cu, net +5V
- removed copper zone on B.Cu, net +BATT
- removed copper zone on F.Cu, net +BATT
- removed copper zone on B.Cu, net -BATT
- removed copper zone on F.Cu, net -BATT
- removed copper zone on B.Cu, net /Cell1
- removed copper zone on F.Cu, net /Cell1
- removed copper zone on B.Cu, net Net-(BT3--)
- removed copper zone on F.Cu, net Net-(BT3--)
- removed copper zone on B.Cu, net Net-(BT5--)
- removed copper zone on F.Cu, net Net-(BT5--)
- removed copper zone on B.Cu, net Net-(Q1-S)
Other:
- board size 514.8 x 95 mm -> 338 x 140 mm
- board text added: "SYM"
- board text removed: "Batt+"
- board text removed: "Batt-"
