File: MotorDriverDualHalfBridge.kicad_sch (KiCad schematic)
At the start: 42 parts, among them J3 Batt+, J3 Batt-, J3 Motor Bottom Connection, J3 Motor Middle Connection, J3 Motor Upper Connection, J6 Conn_01x04, Q1 IAUA250N04S6N005, Q2 IAUA250N04S6N005, U1 2ED21824S06J, U2 EL817, U3 EL817

Commit message: Motor Driver V1.1
Parts:
- removed C20: 100uF, Capacitor_SMD:CP_Elec_6.3x5.4_Nichicon, symbol Device:C_Polarized_Small_US
- removed J6 (x2): Conn_01x04, Library:MOLEX_2078430004_L1NK_250_4-PIN, symbol Connector_Generic:Conn_01x04
- removed R1 (x4): R_{DT}, Resistor_THT:R_Axial_DIN0207_L6.3mm_D2.5mm_P10.16mm_Horizontal, symbol Device:R_Small
- removed U2, U3: EL817, Package_DIP:DIP-4_W7.62mm, symbol Isolator:EL817
- added C1: 0.1uF, Capacitor_SMD:C_0603_1608Metric_Pad1.08x0.95mm_HandSolder, symbol Device:C_Small
- added C1: 100uF, Capacitor_SMD:C_Elec_5x5.8, symbol Device:C_Small
- added C1: 22uF, Capacitor_SMD:CP_Elec_5x5.8, symbol Device:C_Small
- added J7: Conn_01x02, Connector_JST:JST_EH_B2B-EH-A_1x02_P2.50mm_Vertical, symbol Connector_Generic:Conn_01x02
- added R1: R_{DT}, Resistor_THT:R_Axial_DIN0207_L6.3mm_D2.5mm_P10.16mm_Horizontal, symbol Device:R_Small
- added R1: 1.8k, Resistor_THT:R_Axial_DIN0207_L6.3mm_D2.5mm_P10.16mm_Horizontal, symbol Device:R_Small
- added U2: ~, Library:I3A4W005A150V001R, symbol SymbolLibrary:U?
- added U4: LM358, Package_DIP:DIP-8_W7.62mm_LongPads, symbol Amplifier_Operational:LM358
- added U5: EL817, Package_DIP:DIP-4_W7.62mm, symbol Isolator:EL817
- C1, C4, C5, R4, R5: now not fitted
Connections:
- net GND is gone; now on net GNDPWR: C1.2, C2.2, JP1.1 (A), R1.2, U1. (V_{SS}), U1.5 (COM)
- net H_{IN}_{_ISO} is gone; now on net H_{IN}: U1.1 (HIN)
- net L_{IN}_{_ISO} is gone; now on net L_{IN}: U1.2 (LIN)
- net +12V: now also C1.1, C1.1, U2.7 (SENSE), U2.8 (V_{OUT}+), U4.8 (V+), U5.4
- net +BATT: now also C1.1, U2.1 (V_{IN+})
- net GNDPWR: now also C1.2, C1.2, C1.2, R1.1, R1.2, U2.2 (ON/OFF), U2.3 (V_{IN-}), U2.4 (V_{OUT}-), U4.3 (+), U4.4 (V-), U4.6 (-)
- net H_{IN}: now also U4.1
- net L_{IN}: now also U4.7
- new net: R1.1, U4.2 (-), U4.5 (+), U5.3
- new net: R1.2, U2.6 (TRIM)
- new net MotorDrive +: J7.1 (Pin_1), U5.1
- new net MotorDriver -: J7.2 (Pin_2), U5.2
Other:
- note removed: "20V Max"
- moved on the sheet: C16, C17, C18, C2, C3, J3, JP1, Q1, Q2, R1, R2, R3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
